Commit message: Checkpoint: Gazebo + URDF + ros2_control wiring (controllers not stabilized)

File: src/rover_description/urdf/rover.urdf (robot description, URDF)
Before this commit: robot rover, 3 links, 2 joints
Links:
- added link lidar_link
- link base_link: mass 10.0 -> 10; geometry collision box size=0.6 0.4 0.2; visual box size=0.6 0.4 0.2
- link left_wheel: mass 1.0 -> 1; geometry collision cylinder length=0.05 radius=0.08; visual cylinder length=0.05 radius=0.08
- link right_wheel: mass 1.0 -> 1; geometry collision cylinder length=0.05 radius=0.08; visual cylinder length=0.05 radius=0.08
Joints:
- added joint lidar_joint: type fixed, parent base_link, child lidar_link, origin xyz=0.25 0 0.15
- joint left_wheel_joint: axis 0 0 1 -> 0 1 0; origin xyz=0 0.15 0 rpy=0 1.5708 0 -> xyz=0 0.2 -0.1
- joint right_wheel_joint: axis 0 0 1 -> 0 1 0; origin xyz=0 -0.15 0 rpy=0 1.5708 0 -> xyz=0 -0.2 -0.1
